File: pcb/KiBot-CICD-Template.kicad_sch (KiCad schematic)
At the start: 1 part

Commit message: modified kicad data
Parts:
- R1: value (none) -> R; footprint (none) -> Resistor_SMD:R_0603_1608Metric
Other:
- moved on the sheet: R1
Changed lines of the file:
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@@
     (comment 4 "CERN Open Hardware Licence v2.0")
   )
-  (wire (pts (xy 99.06 97.79) (xy 99.06 119.38))
+  (wire (pts (xy 104.14 88.9) (xy 104.14 110.49))
     (stroke (width 0) (type default) (color 0 0 0 0))
   )
-  (wire (pts (xy 99.06 119.38) (xy 109.22 119.38))
+  (wire (pts (xy 104.14 110.49) (xy 114.3 110.49))
     (stroke (width 0) (type default) (color 0 0 0 0))
   )
-  (wire (pts (xy 109.22 106.68) (xy 109.22 97.79))
+  (wire (pts (xy 114.3 97.79) (xy 114.3 88.9))
     (stroke (width 0) (type default) (color 0 0 0 0))
   )
-  (wire (pts (xy 109.22 97.79) (xy 99.06 97.79))
+  (wire (pts (xy 114.3 88.9) (xy 104.14 88.9))
     (stroke (width 0) (type default) (color 0 0 0 0))
   )
-  (wire (pts (xy 109.22 119.38) (xy 109.22 114.3))
+  (wire (pts (xy 114.3 110.49) (xy 114.3 105.41))
     (stroke (width 0) (type default) (color 0 0 0 0))
   )
@@
     )
   )
-  (symbol (lib_id "Device:R") (at 109.22 110.49 0) (unit 1)
+  (symbol (lib_id "Device:R") (at 114.3 101.6 0) (unit 1)
     (in_bom yes) (on_board yes) (fields_autoplaced)
-    (property "Reference" "R1" (id 0) (at 111.76 109.2199 0)
+    (property "Reference" "R1" (id 0) (at 116.84 100.3299 0)
       (effects (font (size 1.27 1.27)) (justify left))
     )
-    (property "Value" "" (id 1) (at 111.76 111.7599 0)
+    (property "Value" "R" (id 1) (at 116.84 102.8699 0)
       (effects (font (size 1.27 1.27)) (justify left))
     )
-    (property "Footprint" "" (id 2) (at 107.442 110.49 90)
+    (property "Footprint" "Resistor_SMD:R_0603_1608Metric" (id 2) (at 112.522 101.6 90)
       (effects (font (size 1.27 1.27)) hide)
     )
-    (property "Datasheet" "~" (id 3) (at 109.22 110.49 0)
+    (property "Datasheet" "~" (id 3) (at 114.3 101.6 0)
       (effects (font (size 1.27 1.27)) hide)
     )
-    (property "Variant" "DNP" (id 4) (at 109.22 110.49 0)
+    (property "Variant" "DNP" (id 4) (at 114.3 101.6 0)
       (effects (font (size 1.27 1.27)) hide)
     )
@@
     )
     (path "/5f38bdb2-3657-474e-8e86-d6bb0b298110"
-      (reference "R1") (unit 1) (value "R") (footprint "")
+      (reference "R1") (unit 1) (value "R") (footprint "Resistor_SMD:R_0603_1608Metric")
     )
   )
